Commit message: ur5 rerun viz suite for deligrasp, converted from droid/franka

File: viz/ur_description/urdf/ur5.urdf (robot description, URDF)
Before this commit: robot ur5_robot, 11 links, 10 joints
Links:
- link base_link_inertia: geometry collision mesh filename=/home/will/MAGPIE/viz/ur_description/meshes/ur5/collision/b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; visual mesh filename=/home/will/MAGPIE/viz/ur_description/meshes/ur5/visual/base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
- link forearm_link: geometry collision mesh filename=/home/will/MAGPIE/viz/ur_description/meshes/ur5/collision/f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; visual mesh filename=/home/will/MAGPIE/viz/ur_description/meshes/ur5/visual/fore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
- link shoulder_link: geometry collision mesh filename=/home/will/MAGPIE/viz/ur_description/meshes/ur5/collision/s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; visual mesh filename=/home/will/MAGPIE/viz/ur_description/meshes/ur5/visual/shou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
- link upper_arm_link: geometry collision mesh filename=/home/will/MAGPIE/viz/ur_description/meshes/ur5/collision/u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; visual mesh filename=/home/will/MAGPIE/viz/ur_description/meshes/ur5/visual/uppe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
- link wrist_1_link: geometry collision mesh filename=/home/will/MAGPIE/viz/ur_description/meshes/ur5/collision/w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; visual mesh filename=/home/will/MAGPIE/viz/ur_description/meshes/ur5/visual/wris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
- link wrist_2_link: geometry collision mesh filename=/home/will/MAGPIE/viz/ur_description/meshes/ur5/collision/w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; visual mesh filename=/home/will/MAGPIE/viz/ur_description/meshes/ur5/visual/wris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
- link wrist_3_link: geometry collision mesh filename=/home/will/MAGPIE/viz/ur_description/meshes/ur5/collision/w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; visual mesh filename=/home/will/MAGPIE/viz/ur_description/meshes/ur5/visual/wris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
